File: mechanical-keyboard-pcb.sch (KiCad schematic (older format))
At the start: 152 parts, among them U0 MX-LED, U1 MX-LED, U10 MX-LED, U11 MX-LED, U12 MX-LED, U13 MX-LED, U14 MX-LED, U15 MX-LED, U16 MX-LED, U17 MX-LED, U18 MX-LED, U19 MX-LED, U2 MX-LED, U20 MX-LED, U21 MX-LED, U22 MX-LED, U23 MX-LED, U24 MX-LED, U25 MX-LED, U26 MX-LED, U27 MX-LED, U28 MX-LED, U29 MX-LED, U3 MX-LED, U30 MX-LED, U31 MX-LED, U32 MX-LED, U33 MX-LED, U34 MX-LED, U35 MX-LED, U36 MX-LED, U37 MX-LED, U38 MX-LED, U39 MX-LED, U4 MX-LED, U40 MX-LED, U41 MX-LED, U42 MX-LED, U43 MX-LED, U44 MX-LED, U45 MX-LED, U46 MX-LED, U47 MX-LED, U48 MX-LED, U49 MX-LED, U5 MX-LED, U50 MX-LED, U51 MX-LED, U52 MX-LED, U53 MX-LED, U54 MX-LED, U55 MX-LED, U56 MX-LED, U57 MX-LED, U58 MX-LED, U59 MX-LED, U6 MX-LED, U60 MX-LED, U61 MX-LED, U62 MX-LED, U63 MX-LED, U64 MX-LED, U65 MX-LED, U66 MX-LED, U67 MX-LED, U7 MX-LED, U8 MX-LED, U9 MX-LED

Commit message: Keyboard schematic with individually addressable RGB LEDs
Parts:
- removed C?: C_Small, symbol Device:C_Small
- removed C? (x2): 22 pF, symbol Device:C_Small
- removed D? (x68): D_Small, symbol Device:D_Small
- removed R? (x2): 10k, symbol Device:R_Small
- removed R? (x2): 22, symbol Device:R_Small
- removed SW?: SW_Push, symbol Switch:SW_Push
- removed U0, U1, U10, U11, U12, U13, U14, U15, U16, U17, U18, U19, U2, U20, U21, U22, U23, U24, U25, U26, U27, U28, U29, U3, U30, U31, U32, U33, U34, U35, U36, U37, U38, U39, U4, U40, U41, U42, U43, U44, U45, U46, U47, U48, U49, U5, U50, U51, U52, U53, U54, U55, U56, U57, U58, U59, U6, U60, U61, U62, U63, U64, U65, U66, U67, U7, U8, U9: MX-LED, symbol MX_Alps_Hybrid:MX-LED
- removed U?: ATmega32U4-AU, Package_QFP:TQFP-44_10x10mm_P0.8mm, symbol MCU_Microchip_ATmega:ATmega32U4-AU
- removed Y?: 16MHz, symbol Device:Crystal_GND24_Small
- added C? (x3): 0.1 uF, symbol Device:C_Small
- added C?: C_Small, symbol Device:C_Small
- added C? (x2): 22 pF, symbol Device:C_Small
- added R? (x3): 20k, symbol Device:R_Small
- added R? (x9): 4.7k, symbol Device:R_Small
- added R? (x3): 100k, symbol Device:R_Small
- added R? (x2): 10k, symbol Device:R_Small
- added R? (x2): 22, symbol Device:R_Small
- added SW?: SW_Push, symbol Switch:SW_Push
- added U? (x3): IS31FL3731-QF, Package_DFN_QFN:QFN-28-1EP_4x4mm_P0.4mm_EP2.3x2.3mm, symbol Driver_LED:IS31FL3731-QF
- added U? (x68): MX-RGB, symbol keyboard:MX-RGB
- added U?: AT90USB1286-AU, Package_QFP:TQFP-64_14x14mm_P0.8mm, symbol MCU_Microchip_AVR:AT90USB1286-AU
- added Y?: 16MHz, symbol Device:Crystal_GND24_Small
Connections:
- net +5V is gone; now on net VCC: C?.1, C?.1, C?.1, C?.1, F?.1
- net COL0: now also U?.1 (COL), U?.1 (COL), U?.1 (COL), U?.1 (COL), U?.1 (COL), U?.1 (COL), U?.1 (COL), U?.1 (COL), U?.1 (COL), U?.1 (COL)
- net COL1: now also U?.1 (COL), U?.1 (COL), U?.1 (COL), U?.1 (COL), U?.1 (COL), U?.1 (COL), U?.1 (COL), U?.1 (COL), U?.1 (COL), U?.1 (COL)
- net COL2: now also U?.1 (COL), U?.1 (COL), U?.1 (COL), U?.1 (COL), U?.1 (COL), U?.1 (COL), U?.1 (COL), U?.1 (COL), U?.1 (COL), U?.1 (COL)
- net COL3: now also U?.1 (COL), U?.1 (COL), U?.1 (COL), U?.1 (COL), U?.1 (COL), U?.1 (COL), U?.1 (COL), U?.1 (COL), U?.1 (COL), U?.1 (COL)
- net COL4: now also U?.1 (COL), U?.1 (COL), U?.1 (COL), U?.1 (COL), U?.1 (COL), U?.1 (COL), U?.1 (COL), U?.1 (COL), U?.1 (COL), U?.1 (COL)
- net COL5: now also U?.1 (COL), U?.1 (COL), U?.1 (COL), U?.1 (COL), U?.1 (COL), U?.1 (COL), U?.1 (COL), U?.1 (COL)
- net COL6: now also U?.1 (COL), U?.1 (COL), U?.1 (COL), U?.1 (COL), U?.1 (COL), U?.1 (COL), U?.1 (COL), U?.1 (COL)
- net D+: now also R?.2
- net D-: now also R?.2
- net GND: now also C?.1, C?.1, C?.1, C?.1, C?.1, C?.2, R?.1, R?.2, R?.2, R?.2, R?.2, R?.2, R?.2, R?.2, R?.2, R?.2, R?.2, R?.2, R?.2, R?.2, R?.2, R?.2, SW?.1, U?.18 (AD), U?.18 (AD), U?.18 (AD), U?.22 (GND), U?.29 (GND), U?.29 (GND), U?.29 (GND), U?.5 (GND), U?.5 (GND), U?.5 (GND), U?.53 (GND), U?.6 (UGND), U?.63 (GND), Y?.2, Y?.4
- net ROW0: now also U?.2 (ROW), U?.2 (ROW), U?.2 (ROW), U?.2 (ROW), U?.2 (ROW), U?.2 (ROW), U?.2 (ROW), U?.2 (ROW)
- net ROW1: now also U?.2 (ROW), U?.2 (ROW), U?.2 (ROW), U?.2 (ROW), U?.2 (ROW), U?.2 (ROW), U?.2 (ROW)
- net ROW2: now also U?.2 (ROW), U?.2 (ROW), U?.2 (ROW), U?.2 (ROW), U?.2 (ROW), U?.2 (ROW), U?.2 (ROW), U?.2 (ROW)
- net ROW3: now also U?.2 (ROW), U?.2 (ROW), U?.2 (ROW), U?.2 (ROW), U?.2 (ROW), U?.2 (ROW), U?.2 (ROW)
- net ROW4: now also U?.2 (ROW), U?.2 (ROW), U?.2 (ROW), U?.2 (ROW), U?.2 (ROW), U?.2 (ROW), U?.2 (ROW)
- net ROW5: now also U?.2 (ROW), U?.2 (ROW), U?.2 (ROW), U?.2 (ROW), U?.2 (ROW), U?.2 (ROW), U?.2 (ROW)
- net ROW6: now also U?.2 (ROW), U?.2 (ROW), U?.2 (ROW), U?.2 (ROW), U?.2 (ROW), U?.2 (ROW), U?.2 (ROW)
- net ROW7: now also U?.2 (ROW), U?.2 (ROW), U?.2 (ROW), U?.2 (ROW), U?.2 (ROW), U?.2 (ROW), U?.2 (ROW)
- net VCC: now also R?.1, U?.2 (VCC), U?.2 (VCC), U?.2 (VCC), U?.21 (VCC), U?.3 (UVCC), U?.52 (VCC), U?.64 (AVCC); no longer F?.2, USB?.5 (VBUS)
- new net: C?.2, U?.16 (C_FILT) (x3)
- new net: R?.1, U?.6 (R_EXT) (x3)
- new net: R?.2, SW?.2, U?.20 (~RESET)
- new net: U?.23 (XTAL2), Y?.3
- new net: C?.1, U?.24 (XTAL1), Y?.1
- new net: R?.1, U?.4 (D-)
- new net: R?.2, U?.43 (PE2/~HWB)
- new net: R?.1, U?.5 (D+)
- new net: C?.2, U?.7 (UCAP)
- new net COL7: U?.1 (COL), U?.1 (COL)
- new net DRV0_INTB: R?.1, U?.4 (~INTB)
- new net DRV0_SCL: R?.1, U?.20 (SCL)
- new net DRV0_SDA: R?.1, U?.19 (SDA)
- new net DRV0_SDB: R?.1, U?.3 (~SDB)
- new net DRV1_INTB: R?.1, U?.4 (~INTB)
- new net DRV1_SCL: R?.1, U?.20 (SCL)
- new net DRV1_SDA: R?.1, U?.19 (SDA)
- new net DRV1_SDB: R?.1, U?.3 (~SDB)
- new net DRV2_INTB: R?.1, U?.4 (~INTB)
- new net DRV2_SCL: R?.1, U?.20 (SCL)
- new net DRV2_SDA: R?.1, U?.19 (SDA)
- new net DRV2_SDB: R?.1, U?.3 (~SDB)
- new net LED0: U?.3 (R), U?.3 (R), U?.3 (R), U?.3 (R), U?.3 (R), U?.3 (R), U?.3 (R), U?.3 (R), U?.~ (G)
- new net LED1: U?.~ (G), U?.~ (G), U?.~ (G), U?.~ (G), U?.~ (G), U?.~ (G), U?.~ (G), U?.~ (G), U?.~ (G)
- new net LED10: U?.~ (G), U?.~ (G), U?.~ (G), U?.~ (G), U?.~ (G), U?.~ (G), U?.~ (G), U?.~ (G)
- new net LED11: U?.4 (B), U?.4 (B), U?.4 (B), U?.4 (B), U?.4 (B), U?.~ (G), U?.~ (G), U?.~ (G)
- new net LED12: U?.4 (B), U?.4 (B), U?.~ (G), U?.~ (G)
- new net LED13: U?.~ (G), U?.~ (G)
- new net LED14: U?.4 (B), U?.~ (G), U?.~ (G)
- new net LED15: U?.4 (B), U?.4 (B), U?.4 (B), U?.4 (B), U?.4 (B), U?.4 (B), U?.~ (G), U?.~ (G)
- new net LED16: U?.~ (G), U?.~ (G), U?.~ (G), U?.~ (G), U?.~ (G), U?.~ (G), U?.~ (G), U?.~ (G)
- new net LED17: U?.3 (R), U?.3 (R), U?.3 (R), U?.3 (R), U?.3 (R), U?.3 (R), U?.3 (R)
- new net LED18: U?.3 (R), U?.3 (R), U?.3 (R), U?.3 (R), U?.3 (R), U?.3 (R), U?.3 (R), U?.3 (R), U?.~ (G)
- new net LED19: U?.~ (G), U?.~ (G), U?.~ (G), U?.~ (G), U?.~ (G), U?.~ (G), U?.~ (G), U?.~ (G), U?.~ (G)
- new net LED2: U?.4 (B), U?.4 (B), U?.4 (B), U?.4 (B), U?.4 (B), U?.4 (B), U?.~ (G), U?.~ (G), U?.~ (G)
- new net LED20: U?.4 (B), U?.4 (B), U?.4 (B), U?.4 (B), U?.4 (B), U?.4 (B), U?.~ (G), U?.~ (G), U?.~ (G)
- new net LED21: U?.4 (B), U?.4 (B), U?.~ (G), U?.~ (G)
- new net LED22: U?.~ (G), U?.~ (G)
- new net LED23: U?.4 (B), U?.4 (B), U?.~ (G), U?.~ (G)
- new net LED24: U?.4 (B), U?.4 (B), U?.4 (B), U?.4 (B), U?.4 (B), U?.4 (B), U?.~ (G), U?.~ (G), U?.~ (G)
- new net LED25: U?.~ (G), U?.~ (G), U?.~ (G), U?.~ (G), U?.~ (G), U?.~ (G), U?.~ (G), U?.~ (G), U?.~ (G)
- new net LED26: U?.3 (R), U?.3 (R), U?.3 (R), U?.3 (R), U?.3 (R), U?.3 (R), U?.3 (R), U?.3 (R), U?.~ (G)
- new net LED27: U?.3 (R), U?.3 (R), U?.3 (R), U?.3 (R), U?.3 (R), U?.3 (R), U?.~ (G)
- new net LED28: U?.~ (G), U?.~ (G), U?.~ (G), U?.~ (G), U?.~ (G), U?.~ (G), U?.~ (G)
- new net LED29: U?.4 (B), U?.4 (B), U?.4 (B), U?.4 (B), U?.~ (G), U?.~ (G), U?.~ (G)
- new net LED3: U?.4 (B), U?.4 (B), U?.~ (G), U?.~ (G)
- new net LED30: U?.4 (B), U?.4 (B), U?.~ (G), U?.~ (G)
- new net LED31: U?.~ (G), U?.~ (G)
- new net LED32: U?.~ (G), U?.~ (G)
- new net LED33: U?.4 (B), U?.4 (B), U?.4 (B), U?.4 (B), U?.4 (B), U?.4 (B), U?.~ (G)
- new net LED34: U?.~ (G), U?.~ (G), U?.~ (G), U?.~ (G), U?.~ (G), U?.~ (G)
- new net LED35: U?.3 (R), U?.3 (R), U?.3 (R), U?.3 (R), U?.3 (R), U?.3 (R)
- new net LED36: U?.3 (R), U?.3 (R), U?.3 (R), U?.3 (R), U?.3 (R), U?.3 (R), U?.3 (R), U?.3 (R), U?.~ (G)
- new net LED37: U?.~ (G), U?.~ (G), U?.~ (G), U?.~ (G), U?.~ (G), U?.~ (G), U?.~ (G), U?.~ (G), U?.~ (G)
- new net LED38: U?.4 (B), U?.4 (B), U?.4 (B), U?.4 (B), U?.4 (B), U?.4 (B), U?.~ (G), U?.~ (G)
- new net LED39: U?.4 (B), U?.4 (B), U?.~ (G)
- new net LED4: U?.~ (G), U?.~ (G)
- new net LED40: U?.~ (G)
- new net LED41: U?.~ (G)
- new net LED42: U?.4 (B), U?.4 (B), U?.~ (G)
- new net LED43: U?.~ (G), U?.~ (G), U?.~ (G)
- new net LED44: U?.3 (R), U?.3 (R), U?.~ (G)
- new net LED5: U?.4 (B), U?.4 (B), U?.~ (G), U?.~ (G)
- new net LED6: U?.4 (B), U?.4 (B), U?.4 (B), U?.4 (B), U?.4 (B), U?.4 (B), U?.~ (G), U?.~ (G), U?.~ (G)
- new net LED7: U?.~ (G), U?.~ (G), U?.~ (G), U?.~ (G), U?.~ (G), U?.~ (G), U?.~ (G), U?.~ (G), U?.~ (G)
- new net LED8: U?.3 (R), U?.3 (R), U?.3 (R), U?.3 (R), U?.3 (R), U?.3 (R), U?.3 (R), U?.3 (R), U?.~ (G)
- new net LED9: U?.3 (R), U?.3 (R), U?.3 (R), U?.3 (R), U?.3 (R), U?.3 (R), U?.3 (R), U?.~ (G)
- new net ROW8: U?.2 (ROW), U?.2 (ROW), U?.2 (ROW), U?.2 (ROW), U?.2 (ROW)
- new net ROW9: U?.2 (ROW), U?.2 (ROW), U?.2 (ROW), U?.2 (ROW), U?.2 (ROW)
- new net VBUS: F?.2, U?.8 (VBUS), USB?.5 (VBUS)
Other:
- moved on the sheet: C?, F?, USB?
